File: dualevse.sch (EAGLE design)
At the start: 54 parts, among them J2 I2C, J3 EXP, Q1 2N2222A, Q2 2N2222A, Q3 2N2222A, Q4 2N2222A, X1 RELAY, X2 CHARGE1, X3 CHARGE2, X4 RS485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

Commit message: Changed some texts
Other:
- note added: "DUAL EVSE v0.9"
- note removed: "DUAL EVSE"
- moved on the sheet: D6, D7, D8, R11, R12, R13, R14, R15, R16, R17, R18, R19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
