File: eagle/dualevse.brd (EAGLE design)
At the start: 70 x 72 mm, 54 parts, among them J2 I2C, J3 EXP, Q1 2N2222A, Q2 2N2222A, Q3 2N2222A, Q4 2N2222A, X1 RELAY, X2 CHARGE1, X3 CHARGE2, X4 RS485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

Commit message: version 0.91
added 2 capacitors
Parts:
- added C8, C9: 22pF, SparkFun-Capacitors:CAP-PTH-2.54
Connections:
- net CP1: now also C9.1
- net CP2: now also C8.1
- net GND: now also C8.2, C9.2
Routing:
- net -12V: track 42.0 -> 118.0 mm, vias 0 -> 5
- net PWM1: track 79.8 -> 125.3 mm
- net RX: track 55.5 -> 80.1 mm, vias 2 -> 1
- net CP_READ2: track 39.1 -> 62.7 mm
- net A: track 35.8 -> 59.4 mm, vias 0 -> 1
- net RELAY2: track 61.7 -> 83.3 mm
- net DIR: track 70.5 -> 87.7 mm, vias 1 -> 0
- net DC_RELAY_1: track 57.9 -> 41.7 mm, vias 0 -> 2
- net PP1: track 28.6 -> 42.8 mm, vias 0 -> 1
- net PP_READ2: track 41.9 -> 49.2 mm, vias 0 -> 1
- net N$10: track 42.2 -> 49.4 mm, vias 2 -> 1
- net +12V: track 140.3 -> 146.2 mm, vias 1 -> 0
- net TX: track 68.0 -> 73.8 mm
- net PP2: track 33.8 -> 39.2 mm, vias 0 -> 2
- net +5V: track 119.6 -> 124.4 mm
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Other:
- board text added: "DUALEVSE v0.91"
- board text removed: "DUALEVSE v0.9"

Commit message: v 0.91a
Parts:
- moved D5 3.81 mm to (31.8, 26.7)
- moved D7 3.81 mm to (48.3, 26.7)
- moved C8 2.54 mm to (48.3, 14.0)
- moved C9 2.54 mm to (31.8, 14.0)
Routing:
- net N$10: track 49.4 -> 107.2 mm
- net PWM1: track 125.3 -> 94.6 mm
- net -12V: track 118.0 -> 95.3 mm, vias 5 -> 2
- net A: track 59.4 -> 36.9 mm, vias 1 -> 0
- net AC_RELAY_1: track 63.2 -> 85.2 mm, vias 0 -> 2
- net N$11: track 39.6 -> 59.7 mm, vias 0 -> 1
- net +5V: track 124.4 -> 144.3 mm
- net DIR: track 87.7 -> 69.6 mm, vias 0 -> 3
- net TX: track 73.8 -> 62.0 mm
- net RELAY1: track 45.9 -> 55.5 mm, vias 2 -> 0
- net PP1: track 42.8 -> 34.3 mm, vias 1 -> 0
- net CP2: track 22.3 -> 30.5 mm
- net PP_READ2: track 49.2 -> 41.9 mm, vias 1 -> 0
- net AC_RELAY_2: track 54.1 -> 61.1 mm
- net CP1: track 24.1 -> 31.0 mm
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